File: STM-32/STM-32.kicad_pcb (KiCad board)
At the start: 4 copper layers, 38 x 45 mm, 43 parts, among them J1 Screw_Terminal_01x02, J2 Conn_02x05_Odd_Even, J3 Conn_01x04, J4 Conn_01x04, J5 USB_B_Micro, Q1 AO3401A, SW1 SW_SPDT, U1 STM32F405RG6, U2 MP2359DJ-LF-Z, U3 USBLC6-2SC6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

Commit message: gnd edited
Connections:
- Q1 pad 1: +5V -> GND
Changed lines of the file:
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@@
 			(layers "F.Cu" "F.Paste" "F.Mask")
 			(roundrect_rratio 0.25)
-			(net 13 "+5V")
+			(net 1 "GND")
 			(pinfunction "G")
 			(pintype "input")
