File: keyboard/keyboard.kicad_pcb (KiCad board)
At the start: 2 copper layers, 439.7 x 109.3 mm, 179 parts, among them U1 RASPBERRY_PI_PICO

Commit message: keyboard design - Routing V1
Parts:
- moved D65 2.39 mm to (261.4, 213.0)
- moved D66 2.39 mm to (280.5, 213.0)
- moved D70 2.39 mm to (356.7, 213.0)
- moved D71 2.39 mm to (392.4, 213.0)
- moved D73 2.39 mm to (475.7, 213.0)
- moved D74 2.39 mm to (494.8, 213.0)
- moved D59 2.39 mm to (99.5, 213.0)
- moved D60 2.39 mm to (154.3, 213.0)
- moved D61 2.39 mm to (185.2, 213.0)
- moved D62 2.39 mm to (204.3, 213.0)
- moved D64 2.39 mm to (242.4, 213.0)
- moved D63 2.39 mm to (223.3, 213.0)
- moved D67 2.39 mm to (299.5, 213.0)
- moved D68 2.39 mm to (318.6, 213.0)
- moved D69 2.39 mm to (337.6, 213.0)
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Connections:
- net Net-(MX1-Pad1) renamed COL0
- D1 pad 1: Net-(D1-K) -> ROW0
- D10 pad 1: Net-(D1-K) -> ROW0
- D11 pad 1: Net-(D1-K) -> ROW0
- D12 pad 1: Net-(D1-K) -> ROW0
- D13 pad 1: Net-(D1-K) -> ROW0
- D14 pad 1: Net-(D1-K) -> ROW0
- D15 pad 1: Net-(D1-K) -> ROW0
- D16 pad 1: Net-(D1-K) -> ROW0
- D17 pad 1: Net-(D1-K) -> ROW0
- D18 pad 1: Net-(D1-K) -> ROW0
- D19 pad 1: Net-(D1-K) -> ROW0
- D2 pad 1: Net-(D1-K) -> ROW0
- D20 pad 1: Net-(D1-K) -> ROW0
- D21 pad 1: Net-(D21-K) -> ROW1
- D22 pad 1: Net-(D21-K) -> ROW1
- D23 pad 1: Net-(D21-K) -> ROW1
- D24 pad 1: Net-(D21-K) -> ROW1
- D25 pad 1: Net-(D21-K) -> ROW1
- D26 pad 1: Net-(D21-K) -> ROW1
- D27 pad 1: Net-(D21-K) -> ROW1
- D28 pad 1: Net-(D21-K) -> ROW1
- D29 pad 1: Net-(D21-K) -> ROW1
- D3 pad 1: Net-(D1-K) -> ROW0
- D30 pad 1: Net-(D21-K) -> ROW1
- D31 pad 1: Net-(D21-K) -> ROW1
- D32 pad 1: Net-(D21-K) -> ROW1
- D33 pad 1: Net-(D21-K) -> ROW1
- D34 pad 1: Net-(D21-K) -> ROW1
- D35 pad 1: Net-(D21-K) -> ROW1
- D36 pad 1: Net-(D21-K) -> ROW1
- D37 pad 1: Net-(D21-K) -> ROW1
- D38 pad 1: Net-(D21-K) -> ROW1
- D39 pad 1: Net-(D21-K) -> ROW1
- D4 pad 1: Net-(D1-K) -> ROW0
- D40 pad 1: Net-(D21-K) -> ROW1
- D41 pad 1: Net-(D41-K) -> ROW2
- D42 pad 1: Net-(D41-K) -> ROW2
- D43 pad 1: Net-(D41-K) -> ROW2
- D44 pad 1: Net-(D41-K) -> ROW2
- D45 pad 1: Net-(D41-K) -> ROW2
- D46 pad 1: Net-(D41-K) -> ROW2
- D47 pad 1: Net-(D41-K) -> ROW2
- D48 pad 1: Net-(D41-K) -> ROW2
- D49 pad 1: Net-(D41-K) -> ROW2
- D5 pad 1: Net-(D1-K) -> ROW0
- D50 pad 1: Net-(D41-K) -> ROW2
- D51 pad 1: Net-(D41-K) -> ROW2
- D52 pad 1: Net-(D41-K) -> ROW2
- D53 pad 1: Net-(D41-K) -> ROW2
- D54 pad 1: Net-(D41-K) -> ROW2
- D55 pad 1: Net-(D41-K) -> ROW2
- D56 pad 1: Net-(D41-K) -> ROW2
- D57 pad 1: Net-(D41-K) -> ROW2
- D58 pad 1: Net-(D41-K) -> ROW2
- D59 pad 1: Net-(D59-K) -> ROW3
- D6 pad 1: Net-(D1-K) -> ROW0
- D60 pad 1: Net-(D59-K) -> ROW3
- D61 pad 1: Net-(D59-K) -> ROW3
- D62 pad 1: Net-(D59-K) -> ROW3
- D63 pad 1: Net-(D59-K) -> ROW3
- D64 pad 1: Net-(D59-K) -> ROW3
- D65 pad 1: Net-(D59-K) -> ROW3
- D66 pad 1: Net-(D59-K) -> ROW3
- D67 pad 1: Net-(D59-K) -> ROW3
- D68 pad 1: Net-(D59-K) -> ROW3
- D69 pad 1: Net-(D59-K) -> ROW3
- D7 pad 1: Net-(D1-K) -> ROW0
- D70 pad 1: Net-(D59-K) -> ROW3
- D71 pad 1: Net-(D59-K) -> ROW3
- D72 pad 1: Net-(D59-K) -> ROW3
- D73 pad 1: Net-(D59-K) -> ROW3
- D74 pad 1: Net-(D59-K) -> ROW3
- D75 pad 1: Net-(D75-K) -> ROW4
- D76 pad 1: Net-(D59-K) -> ROW3
- D77 pad 1: Net-(D75-K) -> ROW4
- D78 pad 1: Net-(D75-K) -> ROW4
- D79 pad 1: Net-(D75-K) -> ROW4
- D8 pad 1: Net-(D1-K) -> ROW0
- D80 pad 1: Net-(D75-K) -> ROW4
- D81 pad 1: Net-(D75-K) -> ROW4
- D82 pad 1: Net-(D75-K) -> ROW4
- D83 pad 1: Net-(D75-K) -> ROW4
- D84 pad 1: Net-(D75-K) -> ROW4
- D85 pad 1: Net-(D75-K) -> ROW4
- D86 pad 1: Net-(D75-K) -> ROW4
- D87 pad 1: Net-(D75-K) -> ROW4
- D88 pad 1: Net-(D75-K) -> ROW4
- D89 pad 1: Net-(D75-K) -> ROW4
- D9 pad 1: Net-(D1-K) -> ROW0
- MX10 pad 1: Net-(MX10-Pad1) -> COL9
- MX11 pad 1: Net-(MX11-Pad1) -> COL10
- MX12 pad 1: Net-(MX12-Pad1) -> COL11
- MX13 pad 1: Net-(MX13-Pad1) -> COL12
- MX14 pad 1: Net-(MX14-Pad1) -> COL13
- MX15 pad 1: Net-(MX15-Pad1) -> COL14
- MX16 pad 1: Net-(MX16-Pad1) -> COL15
- MX17 pad 1: Net-(MX17-Pad1) -> COL16
- MX18 pad 1: Net-(MX18-Pad1) -> COL17
- MX19 pad 1: Net-(MX19-Pad1) -> COL18
- MX2 pad 1: Net-(MX2-Pad1) -> COL1
- MX20 pad 1: Net-(MX20-Pad1) -> COL19
- MX22 pad 1: Net-(MX2-Pad1) -> COL1
- MX23 pad 1: Net-(MX23-Pad1) -> COL2
- MX24 pad 1: Net-(MX24-Pad1) -> COL3
- MX25 pad 1: Net-(MX25-Pad1) -> COL4
- MX26 pad 1: Net-(MX26-Pad1) -> COL5
- MX27 pad 1: Net-(MX27-Pad1) -> COL6
- MX28 pad 1: Net-(MX28-Pad1) -> COL7
- MX29 pad 1: Net-(MX29-Pad1) -> COL8
- MX3 pad 1: Net-(MX23-Pad1) -> COL2
- MX30 pad 1: Net-(MX10-Pad1) -> COL9
- MX31 pad 1: Net-(MX11-Pad1) -> COL10
- MX32 pad 1: Net-(MX12-Pad1) -> COL11
- MX33 pad 1: Net-(MX13-Pad1) -> COL12
- MX34 pad 1: Net-(MX14-Pad1) -> COL13
- MX35 pad 1: Net-(MX15-Pad1) -> COL14
- MX36 pad 1: Net-(MX16-Pad1) -> COL15
- MX37 pad 1: Net-(MX17-Pad1) -> COL16
- MX38 pad 1: Net-(MX18-Pad1) -> COL17
- MX39 pad 1: Net-(MX19-Pad1) -> COL18
- MX4 pad 1: Net-(MX24-Pad1) -> COL3
- MX40 pad 1: Net-(MX20-Pad1) -> COL19
- MX42 pad 1: Net-(MX2-Pad1) -> COL1
- MX43 pad 1: Net-(MX23-Pad1) -> COL2
- MX44 pad 1: Net-(MX24-Pad1) -> COL3
- MX45 pad 1: Net-(MX25-Pad1) -> COL4
- MX46 pad 1: Net-(MX26-Pad1) -> COL5
- MX47 pad 1: Net-(MX27-Pad1) -> COL6
- MX48 pad 1: Net-(MX28-Pad1) -> COL7
- MX49 pad 1: Net-(MX29-Pad1) -> COL8
- MX5 pad 1: Net-(MX25-Pad1) -> COL4
- MX50 pad 1: Net-(MX10-Pad1) -> COL9
- MX51 pad 1: Net-(MX11-Pad1) -> COL10
- MX52 pad 1: Net-(MX12-Pad1) -> COL11
- MX53 pad 1: Net-(MX13-Pad1) -> COL12
- MX54 pad 1: Net-(MX14-Pad1) -> COL13
- MX55 pad 1: Net-(MX16-Pad1) -> COL15
- MX56 pad 1: Net-(MX17-Pad1) -> COL16
- MX57 pad 1: Net-(MX18-Pad1) -> COL17
- MX58 pad 1: Net-(MX19-Pad1) -> COL18
- MX6 pad 1: Net-(MX26-Pad1) -> COL5
- MX60 pad 1: Net-(MX2-Pad1) -> COL1
- MX61 pad 1: Net-(MX23-Pad1) -> COL2
- MX62 pad 1: Net-(MX24-Pad1) -> COL3
- MX63 pad 1: Net-(MX25-Pad1) -> COL4
- MX64 pad 1: Net-(MX26-Pad1) -> COL5
- MX65 pad 1: Net-(MX27-Pad1) -> COL6
- MX66 pad 1: Net-(MX28-Pad1) -> COL7
- MX67 pad 1: Net-(MX29-Pad1) -> COL8
- MX68 pad 1: Net-(MX10-Pad1) -> COL9
- MX69 pad 1: Net-(MX11-Pad1) -> COL10
- MX7 pad 1: Net-(MX27-Pad1) -> COL6
- MX70 pad 1: Net-(MX12-Pad1) -> COL11
- MX71 pad 1: Net-(MX14-Pad1) -> COL13
- MX72 pad 1: Net-(MX17-Pad1) -> COL16
- MX73 pad 1: Net-(MX18-Pad1) -> COL17
- MX74 pad 1: Net-(MX19-Pad1) -> COL18
- MX75 pad 1: Net-(MX20-Pad1) -> COL19
- MX76 pad 1: Net-(MX15-Pad1) -> COL14
- MX78 pad 1: Net-(MX2-Pad1) -> COL1
- MX79 pad 1: Net-(MX23-Pad1) -> COL2
- MX8 pad 1: Net-(MX28-Pad1) -> COL7
- MX80 pad 1: Net-(MX24-Pad1) -> COL3
- MX81 pad 1: Net-(MX27-Pad1) -> COL6
- MX82 pad 1: Net-(MX11-Pad1) -> COL10
- MX83 pad 1: Net-(MX12-Pad1) -> COL11
- MX84 pad 1: Net-(MX13-Pad1) -> COL12
- MX85 pad 1: Net-(MX17-Pad1) -> COL16
- MX86 pad 1: Net-(MX19-Pad1) -> COL18
- MX87 pad 1: Net-(MX14-Pad1) -> COL13
- MX88 pad 1: Net-(MX15-Pad1) -> COL14
- MX89 pad 1: Net-(MX16-Pad1) -> COL15
- MX9 pad 1: Net-(MX29-Pad1) -> COL8
- U1 pad 1: unconnected-(U1-GP0-Pad1) -> COL2
- U1 pad 10: unconnected-(U1-GP7-Pad10) -> COL14
- U1 pad 11: unconnected-(U1-GP8-Pad11) -> COL13
- U1 pad 12: unconnected-(U1-GP9-Pad12) -> COL12
- U1 pad 14: unconnected-(U1-GP10-Pad14) -> COL11
- U1 pad 15: unconnected-(U1-GP11-Pad15) -> COL10
- U1 pad 16: unconnected-(U1-GP12-Pad16) -> COL9
- U1 pad 17: unconnected-(U1-GP13-Pad17) -> COL8
- U1 pad 19: unconnected-(U1-GP14-Pad19) -> COL7
- U1 pad 2: unconnected-(U1-GP1-Pad2) -> COL1
- U1 pad 20: unconnected-(U1-GP15-Pad20) -> COL6
- U1 pad 21: unconnected-(U1-GP16-Pad21) -> ROW3
- U1 pad 22: unconnected-(U1-GP17-Pad22) -> ROW4
- U1 pad 24: unconnected-(U1-GP18-Pad24) -> ROW2
- U1 pad 25: unconnected-(U1-GP19-Pad25) -> ROW1
- U1 pad 26: unconnected-(U1-GP20-Pad26) -> ROW0
- U1 pad 31: unconnected-(U1-GP26_A0-Pad31) -> COL3
- U1 pad 32: unconnected-(U1-GP27_A1-Pad32) -> COL4
- U1 pad 34: unconnected-(U1-GP28_A2-Pad34) -> COL5
- U1 pad 4: unconnected-(U1-GP2-Pad4) -> COL19
- U1 pad 5: unconnected-(U1-GP3-Pad5) -> COL18
- U1 pad 6: unconnected-(U1-GP4-Pad6) -> COL17
- U1 pad 7: unconnected-(U1-GP5-Pad7) -> COL16
- U1 pad 9: unconnected-(U1-GP6-Pad9) -> COL15
Routing:
- net COL19: track 0.00 -> 554.2 mm
- net COL18: track 0.00 -> 532.5 mm
- net COL16: track 0.00 -> 527.0 mm
- net ROW4: track 0.00 -> 511.9 mm, vias 0 -> 14
- net COL15: track 0.00 -> 497.4 mm
- net ROW0: track 0.00 -> 491.7 mm, vias 0 -> 20
- net ROW1: track 0.00 -> 475.8 mm, vias 0 -> 20
- net COL14: track 0.00 -> 472.4 mm
- net ROW3: track 0.00 -> 471.3 mm, vias 0 -> 17
- net COL13: track 0.00 -> 461.1 mm
- net ROW2: track 0.00 -> 456.9 mm, vias 0 -> 18
- net COL12: track 0.00 -> 422.0 mm
- net COL11: track 0.00 -> 382.0 mm
- net COL10: track 0.00 -> 351.2 mm
- net COL9: track 0.00 -> 324.6 mm
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