File: keyboard/keyboard.kicad_sch (KiCad schematic)
At the start: 179 parts, among them U1 RASPBERRY_PI_PICO

Commit message: keyboard design - Routing V1
Connections:
- net ROW3: now reaches D59.1 (K), D60.1 (K), D61.1 (K), D62.1 (K), D63.1 (K), D64.1 (K), D65.1 (K), D66.1 (K), D67.1 (K), D68.1 (K), D69.1 (K), D70.1 (K), D71.1 (K), D72.1 (K), D73.1 (K), D74.1 (K), D76.1 (K)
- net ROW3: now also U1.21 (GP16)
- net COL15: now reaches MX16.1, MX36.1, MX55.1, MX89.1
- net COL15: now also U1.9 (GP6)
- net ROW1: now reaches D21.1 (K), D22.1 (K), D23.1 (K), D24.1 (K), D25.1 (K), D26.1 (K), D27.1 (K), D28.1 (K), D29.1 (K), D30.1 (K), D31.1 (K), D32.1 (K), D33.1 (K), D34.1 (K), D35.1 (K), D36.1 (K), D37.1 (K), D38.1 (K), D39.1 (K), D40.1 (K)
- net ROW1: now also U1.25 (GP19)
- net COL7: now reaches MX28.1, MX48.1, MX66.1, MX8.1
- net COL7: now also U1.19 (GP14)
- net COL9: now reaches MX10.1, MX30.1, MX50.1, MX68.1
- net COL9: now also U1.16 (GP12)
- net ROW2: now reaches D41.1 (K), D42.1 (K), D43.1 (K), D44.1 (K), D45.1 (K), D46.1 (K), D47.1 (K), D48.1 (K), D49.1 (K), D50.1 (K), D51.1 (K), D52.1 (K), D53.1 (K), D54.1 (K), D55.1 (K), D56.1 (K), D57.1 (K), D58.1 (K)
- net ROW2: now also U1.24 (GP18)
- net COL5: now reaches MX26.1, MX46.1, MX6.1, MX64.1
- net COL5: now also U1.34 (GP28_A2)
- net ROW4: now reaches D75.1 (K), D77.1 (K), D78.1 (K), D79.1 (K), D80.1 (K), D81.1 (K), D82.1 (K), D83.1 (K), D84.1 (K), D85.1 (K), D86.1 (K), D87.1 (K), D88.1 (K), D89.1 (K)
- net ROW4: now also U1.22 (GP17)
- net COL13: now reaches MX14.1, MX34.1, MX54.1, MX71.1, MX87.1
- net COL13: now also U1.11 (GP8)
- net ROW0: now reaches D1.1 (K), D10.1 (K), D11.1 (K), D12.1 (K), D13.1 (K), D14.1 (K), D15.1 (K), D16.1 (K), D17.1 (K), D18.1 (K), D19.1 (K), D2.1 (K), D20.1 (K), D3.1 (K), D4.1 (K), D5.1 (K), D6.1 (K), D7.1 (K), D8.1 (K), D9.1 (K)
- net ROW0: now also U1.26 (GP20)
- net COL0: now reaches MX1.1, MX21.1, MX41.1, MX59.1, MX77.1
- net COL10: now reaches MX11.1, MX31.1, MX51.1, MX69.1, MX82.1
- net COL10: now also U1.15 (GP11)
- net COL18: now reaches MX19.1, MX39.1, MX58.1, MX74.1, MX86.1
- net COL18: now also U1.5 (GP3)
- net COL14: now reaches MX15.1, MX35.1, MX76.1, MX88.1
- net COL14: now also U1.10 (GP7)
- net COL2: now reaches U1.1 (GP0)
- net COL2: now also MX23.1, MX3.1, MX43.1, MX61.1, MX79.1
- net COL12: now reaches U1.12 (GP9)
- net COL12: now also MX13.1, MX33.1, MX53.1, MX84.1
- net COL11: now reaches U1.14 (GP10)
- net COL11: now also MX12.1, MX32.1, MX52.1, MX70.1, MX83.1
- net COL8: now reaches U1.17 (GP13)
- net COL8: now also MX29.1, MX49.1, MX67.1, MX9.1
- net COL1: now reaches U1.2 (GP1)
- net COL1: now also MX2.1, MX22.1, MX42.1, MX60.1, MX78.1
- net COL6: now reaches U1.20 (GP15)
- net COL6: now also MX27.1, MX47.1, MX65.1, MX7.1, MX81.1
- net COL3: now reaches U1.31 (GP26_A0)
- net COL3: now also MX24.1, MX4.1, MX44.1, MX62.1, MX80.1
- net COL4: now reaches U1.32 (GP27_A1)
- net COL4: now also MX25.1, MX45.1, MX5.1, MX63.1
- net COL19: now reaches U1.4 (GP2)
- net COL19: now also MX20.1, MX40.1, MX75.1
- net COL17: now reaches U1.6 (GP4)
- net COL17: now also MX18.1, MX38.1, MX57.1, MX73.1
- net COL16: now reaches U1.7 (GP5)
- net COL16: now also MX17.1, MX37.1, MX56.1, MX72.1, MX85.1
